Commit message: Fix: The laser scanner is now actual height of the laser scanner in RViz and Gazebo

File: urdf/barista_robot_model.urdf (robot description, URDF)
Before this commit: robot barista_robot, 16 links, 15 joints
Links:
- added link lidar_ray_link
- link lidar: geometry collision cylinder length=0.048 radius=0.03; visual mesh filename=package://barista_robot_description/meshes/hokuyo_urg_04lx.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 scale=1.0 1.0 1.0
Joints:
- added joint lidar_ray_joint: type fixed, parent lidar, child lidar_ray_link, origin xyz=0 0 0.048 rpy=0 0 0
- joint chassis_joint: origin xyz=0 0 0.0975 rpy=0 0 0 -> xyz=0 0 0 rpy=0 0 0
- joint lidar_joint: origin xyz=0.12 0 0.125 rpy=0 0 0 -> xyz=0.12 0 0.08 rpy=0 0 0

File: urdf/barista_robot_model.xacro (robot description, xacro)
@@ -44,7 +44,6 @@
   <xacro:property name="damping_coefficient" value="0.0"/>
   <xacro:property name="friction_coefficient" value="0.1"/>
-  <xacro:property name="box_laser_scan_width" value="0.035"/>
-  <xacro:property name="box_laser_scan_height" value="0.05"/>
-  <xacro:property name="box_laser_scan_depth" value="0.035"/>
+  <xacro:property name="cylinder_laser_scan_length" value="0.048"/>
+  <xacro:property name="cylinder_laser_scan_radius" value="0.03"/>
   <!-- Define base_link with visual, collision, and inertial properties -->
   <link name="base_link">
@@ -201,17 +200,17 @@
   </xacro:macro>
   <!-- Macro for Sensor LIDAR -->
-  <xacro:macro name="laser_sensor" params="name color width height depth mass parent_link xyz rpy joint_type axis">
+  <xacro:macro name="laser_sensor" params="name color length radius mass parent_link xyz rpy joint_type axis">
     <link name="lidar">
       <visual>
-        <origin rpy="0 0 0" xyz="0 0 -0.05"/>
-        <geometry>
-          <mesh filename="package://barista_robot_description/meshes/hokuyo_urg_04lx.dae"/>
+        <origin rpy="0 0 0" xyz="0 0 0"/>
+        <geometry>
+          <mesh filename="package://barista_robot_description/meshes/hokuyo_urg_04lx.dae" scale="1.0 1.0 1.0"/>
         </geometry>
         <material name="${color}"/>
       </visual>
       <collision>
-        <origin rpy="0 0 0" xyz="0 0 -0.05"/>
-        <geometry>
-          <mesh filename="package://barista_robot_description/meshes/hokuyo_urg_04lx.dae"/>
+        <origin rpy="0 0 0" xyz="0 0 0"/>
+        <geometry>
+          <cylinder length="${length}" radius="${radius}"/>
         </geometry>
       </collision>
@@ -220,10 +219,10 @@
         <origin xyz="0 0 0"/>
         <inertia
-          ixx="${(1.0/12.0) * mass * (height * height + depth * depth)}"
+          ixx="${(1.0/12.0) * mass * (3.0 * (radius * radius) + (length * length))}"
           ixy="0.0"
           ixz="0.0"
-          iyy="${(1.0/12.0) * mass * (width * width + depth * depth)}"
+          iyy="${(1.0/12.0) * mass * (3.0 * (radius * radius) + (length * length))}"
           iyz="0.0"
-          izz="${(1.0/12.0) * mass * (width * width + height * height)}"/>
+          izz="${(1.0/2.0) * mass * (radius * radius)}"/>
       </inertial>
     </link>
@@ -233,12 +232,19 @@
       <child link="${name}"/>
     </joint>
+    <!-- Ray frame link -->
+    <link name="${name}_ray_link"/>
+    <joint name="${name}_ray_joint" type="fixed">
+      <origin xyz="0 0 ${length}" rpy="0 0 0"/>
+      <parent link="${name}"/>
+      <child link="${name}_ray_link"/>
+    </joint>
     <!-- Laser Sensor Plugin -->
-    <gazebo reference="${name}">
-      <sensor name="sensor_ray" type="ray">
+    <gazebo reference="${name}_ray_link">
+      <sensor name="${name}_sensor" type="ray">
         <pose>0 0 0 0 0 0</pose>
         <ray>
           <scan>
             <horizontal>
-              <samples>200</samples>
+              <samples>720</samples>
               <resolution>1.0</resolution>
               <min_angle>-3.14</min_angle>
@@ -253,11 +259,11 @@
         <visualize>true</visualize>
         <always_on>true</always_on>
-        <update_rate>100.0</update_rate>
-        <plugin name="laser" filename="libgazebo_ros_ray_sensor.so">
+        <update_rate>50.0</update_rate>
+        <plugin name="${name}_gazebo_plugin" filename="libgazebo_ros_ray_sensor.so">
           <ros>
-            <namespace>/barista_robot</namespace>
             <remapping>~/out:=scan</remapping>
           </ros>
           <output_type>sensor_msgs/LaserScan</output_type>
+          <frame_name>${name}_ray_link</frame_name>
         </plugin>
       </sensor>
@@ -271,5 +277,5 @@
                       mass="0.5"
                       parent_link="base_link"
-                      xyz="0 0 0.0975"
+                      xyz="0 0 0"
                       rpy="0 0 0"
                       joint_type="fixed"
@@ -468,10 +474,9 @@
     name="lidar"
     color="Gray"
-    width="${box_laser_scan_width}"
-    height="${box_laser_scan_height}"
-    depth="${box_laser_scan_depth}"
+    length="${cylinder_laser_scan_length}"
+    radius="${cylinder_laser_scan_radius}"
     mass="0.05"
     parent_link="chassis"
-    xyz="0.12 0 0.125"
+    xyz="0.12 0 0.08"
     rpy="0 0 0"
     joint_type="fixed"
