Commit message: Fix typo in worlds file and add small delay in barista_urdf.launch.py

File: urdf/barista_robot_model.xacro (robot description, xacro)
@@ -201,5 +201,5 @@
   <!-- Macro for Sensor LIDAR -->
   <xacro:macro name="laser_sensor" params="name color length radius mass parent_link xyz rpy joint_type axis">
-    <link name="lidar">
+    <link name="${name}">
       <visual>
         <origin rpy="0 0 0" xyz="0 0 0"/>
