Commit message: Fix part 2 of xacro file actual height of the laser scanner in RViz and Gazebo

File: xacro/barista_robot_model.urdf.xacro (robot description, xacro)
@@ -47,7 +47,6 @@
   <xacro:property name="caster_wheel_radius" value="0.02"/>
   <xacro:property name="caster_wheel_length" value="0.01"/>
-  <xacro:property name="box_laser_scan_width" value="0.035"/>
-  <xacro:property name="box_laser_scan_height" value="0.05"/>
-  <xacro:property name="box_laser_scan_depth" value="0.035"/>
+  <xacro:property name="cylinder_laser_scan_length" value="0.048"/>
+  <xacro:property name="cylinder_laser_scan_radius" value="0.03"/>
   <!-- Define base link -->
   <link name="base_link">
@@ -443,15 +442,14 @@
       name="lidar"
       color="Gray"
-      width="${box_laser_scan_width}"
-      height="${box_laser_scan_height}"
-      depth="${box_laser_scan_depth}"
+      length="${cylinder_laser_scan_length}"
+      radius="${cylinder_laser_scan_radius}"
       mass="0.05"
       parent_link="chassis"
-      xyz="0.12 0 0.125"
+      xyz="0.12 0 0.08"
       rpy="0 0 0"
       joint_type="fixed"
       axis="0 0 0"/>
   </xacro:if>
-    <!-- Gazebo Configuration for Laser -->
+  <!-- Gazebo Configuration for Laser -->
   <xacro:if value= "${include_laser}">
     <gazebo reference="lidar">

File: xacro/laser_scanner.xacro (robot description, xacro)
@@ -3,17 +3,18 @@
   <!-- Macro for a Laser Scanner -->
   <!-- Macro for Sensor LIDAR -->
-  <xacro:macro name="laser_scanner" params="name color width height depth mass parent_link xyz rpy joint_type axis">
+   <!-- Macro for Sensor LIDAR -->
+  <xacro:macro name="laser_scanner" params="name color length radius mass parent_link xyz rpy joint_type axis">
     <link name="${name}">
       <visual>
-        <origin rpy="0 0 0" xyz="0 0 -0.05"/>
+        <origin rpy="0 0 0" xyz="0 0 0"/>
         <geometry>
-          <mesh filename="package://barista_robot_description/meshes/hokuyo_urg_04lx.dae"/>
+          <mesh filename="package://barista_robot_description/meshes/hokuyo_urg_04lx.dae" scale="1.0 1.0 1.0"/>
         </geometry>
         <material name="${color}"/>
       </visual>
       <collision>
-        <origin rpy="0 0 0" xyz="0 0 -0.05"/>
+        <origin rpy="0 0 0" xyz="0 0 0"/>
         <geometry>
-          <mesh filename="package://barista_robot_description/meshes/hokuyo_urg_04lx.dae"/>
+          <cylinder length="${length}" radius="${radius}"/>
         </geometry>
       </collision>
@@ -22,10 +23,10 @@
         <origin xyz="0 0 0"/>
         <inertia
-          ixx="${(1.0/12.0) * mass * (height * height + depth * depth)}"
+          ixx="${(1.0/12.0) * mass * (3.0 * (radius * radius) + (length * length))}"
           ixy="0.0"
           ixz="0.0"
-          iyy="${(1.0/12.0) * mass * (width * width + depth * depth)}"
+          iyy="${(1.0/12.0) * mass * (3.0 * (radius * radius) + (length * length))}"
           iyz="0.0"
-          izz="${(1.0/12.0) * mass * (width * width + height * height)}"/>
+          izz="${(1.0/2.0) * mass * (radius * radius)}"/>
       </inertial>
     </link>
@@ -35,12 +36,19 @@
       <child link="${name}"/>
     </joint>
+    <!-- Ray frame link -->
+    <link name="${name}_ray_link"/>
+    <joint name="${name}_ray_joint" type="fixed">
+      <origin xyz="0 0 ${length}" rpy="0 0 0"/>
+      <parent link="${name}"/>
+      <child link="${name}_ray_link"/>
+    </joint>
     <!-- Laser Sensor Plugin -->
-    <gazebo reference="${name}">
-      <sensor name="sensor_ray" type="ray">
+    <gazebo reference="${name}_ray_link">
+      <sensor name="${name}_sensor" type="ray">
         <pose>0 0 0 0 0 0</pose>
         <ray>
           <scan>
             <horizontal>
-              <samples>200</samples>
+              <samples>720</samples>
               <resolution>1.0</resolution>
               <min_angle>-3.14</min_angle>
@@ -55,10 +63,11 @@
         <visualize>true</visualize>
         <always_on>true</always_on>
-        <update_rate>100.0</update_rate>
-        <plugin name="laser" filename="libgazebo_ros_ray_sensor.so">
+        <update_rate>50.0</update_rate>
+        <plugin name="${name}_gazebo_plugin" filename="libgazebo_ros_ray_sensor.so">
           <ros>
-            <remapping>~/out:=/scan</remapping>
+            <remapping>~/out:=scan</remapping>
           </ros>
           <output_type>sensor_msgs/LaserScan</output_type>
+          <frame_name>${name}_ray_link</frame_name>
         </plugin>
       </sensor>

Commit message: Simulation of multiple robots in Rviz and Gazebo

File: xacro/barista_robot_model.urdf.xacro (robot description, xacro)
@@ -1,6 +1,13 @@
 <?xml version="1.0"?>
 <robot xmlns:xacro="http://www.ros.org/wiki/xacro" name="barista_robot">
-  <!-- Arguments -->
+  <!-- Argument -->
+  <xacro:arg name="robot_name" default=""/>
+  <xacro:arg name="color" default=""/>
+  <xacro:arg name="include_laser" default="true"/>
+  <xacro:arg name="plugin_ns" default=""/>
+  <!-- Property -->
   <xacro:property name="include_laser" value="$(arg include_laser)"/>
+  <xacro:property name="robot_name" value="$(arg robot_name)"/>
+  <xacro:property name="color" value="$(arg color)"/>
   <!-- Included tags -->
   <xacro:include filename="$(find barista_robot_description)/xacro/cup_holder_tray.xacro"/>
@@ -59,5 +66,5 @@
         <cylinder length="${body_length}" radius="${body_radius}"/>
       </geometry>
-      <material name="LightNavyBlue"/>
+      <material name="$(arg color)"/>
     </visual>
     <collision>
@@ -79,5 +86,5 @@
   </joint>
   <gazebo reference="chassis">
-    <material>Gazebo/Blue</material>
+    <material>Gazebo/$(arg color)</material>
   </gazebo>
   <!-- Cup Holder Tray -->
@@ -86,5 +93,5 @@
     radius="${cup_holder_tray_radius}"
     length="${cup_holder_tray_length}"
-    material="LightNavyBlue"
+    material="$(arg color)"
     mass="0.2"
     parent_link="chassis"
@@ -94,5 +101,5 @@
     axis="0 0 0"/>
   <gazebo reference="cup_holder_tray">
-    <material>Gazebo/Blue</material>
+    <material>Gazebo/$(arg color)</material>
   </gazebo>
   <!-- Standoff Rods -->
@@ -161,5 +168,5 @@
     mass="0.1"
     parent_link="chassis"
-    xyz="0 -0.12 -0.0623"
+    xyz="0 -0.12 -0.0630"
     rpy="0 1.5708 1.5708"
     joint_type="continuous"
@@ -172,5 +179,5 @@
     mass="0.1"
     parent_link="chassis"
-    xyz="0 0.12 -0.0623"
+    xyz="0 0.12 -0.0630"
     rpy="0 1.5708 1.5708"
     joint_type="continuous"
@@ -178,6 +185,6 @@
   <!-- Gazebo configuration for Wheels -->
   <gazebo reference="wheel_right">
-    <kp>1000000000000000000000000000.0</kp>
-    <kd>1000000000000000000000000000.0</kd>
+    <kp>1000000000.0</kp>
+    <kd>1000000000.0</kd>
     <mu1>0.8</mu1>
     <mu2>0.8</mu2>
@@ -185,6 +192,6 @@
   </gazebo>
   <gazebo reference="wheel_left">
-    <kp>1000000000000000000000000000.0</kp>
-    <kd>1000000000000000000000000000.0</kd>
+    <kp>1000000000.0</kp>
+    <kd>1000000000.0</kd>
     <mu1>0.8</mu1>
     <mu2>0.8</mu2>
@@ -385,6 +392,6 @@
   </gazebo>
   <gazebo reference="front_caster_wheel_pitch_link">
-    <kp>1000000000000000000000000000.0</kp>
-    <kd>1000000000000000000000000000.0</kd>
+    <kp>10000000000.0</kp>
+    <kd>10000000000.0</kd>
     <mu1>0.5</mu1>
     <mu2>0.5</mu2>
@@ -392,6 +399,6 @@
   </gazebo>
   <gazebo reference="back_caster_wheel_pitch_link">
-    <kp>1000000000000000000000000000.0</kp>
-    <kd>1000000000000000000000000000.0</kd>
+    <kp>1000000000.0</kp>
+    <kd>1000000000.0</kd>
     <mu1>0.5</mu1>
     <mu2>0.5</mu2>
@@ -421,4 +428,5 @@
       <ros>
         <remapping>/out:=cmd_vel</remapping>
+        <namespace>$(arg plugin_ns)</namespace>
       </ros>
       <!-- Wheels -->
@@ -434,6 +442,6 @@
       <publish_odom>true</publish_odom>
       <publish_odom_tf>true</publish_odom_tf>
-      <odometry_frame>odom</odometry_frame>
-      <robot_base_frame>base_link</robot_base_frame>
+      <odometry_frame>$(arg robot_name)/odom</odometry_frame>
+      <robot_base_frame>$(arg robot_name)/base_link</robot_base_frame>
     </plugin>
   </gazebo>

File: xacro/wheel.xacro (robot description, xacro)
@@ -4,5 +4,5 @@
   <xacro:property name="joint_effort_limit" value="1000.0"/>
   <xacro:property name="joint_velocity_limit" value="100.0"/>
-  <xacro:property name="damping_coefficient" value="0.0"/>
+  <xacro:property name="damping_coefficient" value="0.02"/>
   <xacro:property name="friction_coefficient" value="0.1"/>
   <!-- Macro for a Wheel Component -->
